Commit message: updated the robot name to atom

File: alphabot_description/urdf/alphabot.xacro (robot description, xacro)
@@ -1,7 +1,7 @@
 <?xml version="1.0" ?>
-<robot name="alphabot" xmlns:xacro="http://www.ros.org/wiki/xacro">
-<xacro:include filename="$(find alphabot_description)/urdf/materials.xacro" />
-<xacro:include filename="$(find alphabot_description)/urdf/alphabot.trans" />
-<xacro:include filename="$(find alphabot_description)/urdf/alphabot.gazebo" />
+<robot name="atom" xmlns:xacro="http://www.ros.org/wiki/xacro">
+<xacro:include filename="$(find atom_description)/urdf/materials.xacro" />
+<xacro:include filename="$(find atom_description)/urdf/atom.trans" />
+<xacro:include filename="$(find atom_description)/urdf/atom.gazebo" />
 <link name="base_link">
   <inertial>
@@ -13,5 +13,5 @@
     <origin xyz="0 0 0" rpy="0 0 0"/>
     <geometry>
-      <mesh filename="file://$(find alphabot_description)/meshes/base_link.stl" scale="0.001 0.001 0.001"/>
+      <mesh filename="file://$(find atom_description)/meshes/base_link.stl" scale="0.001 0.001 0.001"/>
     </geometry>
     <material name="silver"/>
@@ -20,5 +20,5 @@
     <origin xyz="0 0 0" rpy="0 0 0"/>
     <geometry>
-      <mesh filename="file://$(find alphabot_description)/meshes/base_link.stl" scale="0.001 0.001 0.001"/>
+      <mesh filename="file://$(find atom_description)/meshes/base_link.stl" scale="0.001 0.001 0.001"/>
     </geometry>
   </collision>
@@ -33,5 +33,5 @@
     <origin xyz="-0.115 0.134 -0.06" rpy="0 0 0"/>
     <geometry>
-      <mesh filename="file://$(find alphabot_description)/meshes/wheel_clamp_1_1.stl" scale="0.001 0.001 0.001"/>
+      <mesh filename="file://$(find atom_description)/meshes/wheel_clamp_1_1.stl" scale="0.001 0.001 0.001"/>
     </geometry>
     <material name="silver"/>
@@ -40,5 +40,5 @@
     <origin xyz="-0.115 0.134 -0.06" rpy="0 0 0"/>
     <geometry>
-      <mesh filename="file://$(find alphabot_description)/meshes/wheel_clamp_1_1.stl" scale="0.001 0.001 0.001"/>
+      <mesh filename="file://$(find atom_description)/meshes/wheel_clamp_1_1.stl" scale="0.001 0.001 0.001"/>
     </geometry>
   </collision>
@@ -53,5 +53,5 @@
     <origin xyz="-0.23 0.268 0.025" rpy="0 0 0"/>
     <geometry>
-      <mesh filename="file://$(find alphabot_description)/meshes/wheel_1_1.stl" scale="0.001 0.001 0.001"/>
+      <mesh filename="file://$(find atom_description)/meshes/wheel_1_1.stl" scale="0.001 0.001 0.001"/>
     </geometry>
     <material name="silver"/>
@@ -60,5 +60,5 @@
     <origin xyz="-0.23 0.268 0.025" rpy="0 0 0"/>
     <geometry>
-      <mesh filename="file://$(find alphabot_description)/meshes/wheel_1_1.stl" scale="0.001 0.001 0.001"/>
+      <mesh filename="file://$(find atom_description)/meshes/wheel_1_1.stl" scale="0.001 0.001 0.001"/>
     </geometry>
   </collision>
@@ -73,5 +73,5 @@
     <origin xyz="-0.115 -0.134 -0.06" rpy="0 0 0"/>
     <geometry>
-      <mesh filename="file://$(find alphabot_description)/meshes/wheel_clamp_2_1.stl" scale="0.001 0.001 0.001"/>
+      <mesh filename="file://$(find atom_description)/meshes/wheel_clamp_2_1.stl" scale="0.001 0.001 0.001"/>
     </geometry>
     <material name="silver"/>
@@ -80,5 +80,5 @@
     <origin xyz="-0.115 -0.134 -0.06" rpy="0 0 0"/>
     <geometry>
-      <mesh filename="file://$(find alphabot_description)/meshes/wheel_clamp_2_1.stl" scale="0.001 0.001 0.001"/>
+      <mesh filename="file://$(find atom_description)/meshes/wheel_clamp_2_1.stl" scale="0.001 0.001 0.001"/>
     </geometry>
   </collision>
@@ -93,5 +93,5 @@
     <origin xyz="-0.23 -0.268 0.025" rpy="0 0 0"/>
     <geometry>
-      <mesh filename="file://$(find alphabot_description)/meshes/wheel_2_1.stl" scale="0.001 0.001 0.001"/>
+      <mesh filename="file://$(find atom_description)/meshes/wheel_2_1.stl" scale="0.001 0.001 0.001"/>
     </geometry>
     <material name="silver"/>
@@ -100,5 +100,5 @@
     <origin xyz="-0.23 -0.268 0.025" rpy="0 0 0"/>
     <geometry>
-      <mesh filename="file://$(find alphabot_description)/meshes/wheel_2_1.stl" scale="0.001 0.001 0.001"/>
+      <mesh filename="file://$(find atom_description)/meshes/wheel_2_1.stl" scale="0.001 0.001 0.001"/>
     </geometry>
   </collision>
@@ -113,5 +113,5 @@
     <origin xyz="0.115 0.134 -0.06" rpy="0 0 0"/>
     <geometry>
-      <mesh filename="file://$(find alphabot_description)/meshes/wheel_clamp_3_1.stl" scale="0.001 0.001 0.001"/>
+      <mesh filename="file://$(find atom_description)/meshes/wheel_clamp_3_1.stl" scale="0.001 0.001 0.001"/>
     </geometry>
     <material name="silver"/>
@@ -120,5 +120,5 @@
     <origin xyz="0.115 0.134 -0.06" rpy="0 0 0"/>
     <geometry>
-      <mesh filename="file://$(find alphabot_description)/meshes/wheel_clamp_3_1.stl" scale="0.001 0.001 0.001"/>
+      <mesh filename="file://$(find atom_description)/meshes/wheel_clamp_3_1.stl" scale="0.001 0.001 0.001"/>
     </geometry>
   </collision>
@@ -133,5 +133,5 @@
     <origin xyz="0.115 -0.134 -0.06" rpy="0 0 0"/>
     <geometry>
-      <mesh filename="file://$(find alphabot_description)/meshes/wheel_clamp_4_1.stl" scale="0.001 0.001 0.001"/>
+      <mesh filename="file://$(find atom_description)/meshes/wheel_clamp_4_1.stl" scale="0.001 0.001 0.001"/>
     </geometry>
     <material name="silver"/>
@@ -140,5 +140,5 @@
     <origin xyz="0.115 -0.134 -0.06" rpy="0 0 0"/>
     <geometry>
-      <mesh filename="file://$(find alphabot_description)/meshes/wheel_clamp_4_1.stl" scale="0.001 0.001 0.001"/>
+      <mesh filename="file://$(find atom_description)/meshes/wheel_clamp_4_1.stl" scale="0.001 0.001 0.001"/>
     </geometry>
   </collision>
@@ -153,12 +153,12 @@
     <origin xyz="-0.0 -0.0 0.025" rpy="0 0 0"/>
     <geometry>
-      <mesh filename="file://$(find alphabot_description)/meshes/wheel_3_1.stl" scale="0.001 0.001 0.001"/>
-    </geometry>
-    <material name="silver"/>
-  </visual>
-  <collision>
-    <origin xyz="-0.0 -0.0 0.025" rpy="0 0 0"/>
-    <geometry>
-      <mesh filename="file://$(find alphabot_description)/meshes/wheel_3_1.stl" scale="0.001 0.001 0.001"/>
+      <mesh filename="file://$(find atom_description)/meshes/wheel_3_1.stl" scale="0.001 0.001 0.001"/>
+    </geometry>
+    <material name="silver"/>
+  </visual>
+  <collision>
+    <origin xyz="-0.0 -0.0 0.025" rpy="0 0 0"/>
+    <geometry>
+      <mesh filename="file://$(find atom_description)/meshes/wheel_3_1.stl" scale="0.001 0.001 0.001"/>
     </geometry>
   </collision>
@@ -173,12 +173,12 @@
     <origin xyz="-0.0 -0.0 0.025" rpy="0 0 0"/>
     <geometry>
-      <mesh filename="file://$(find alphabot_description)/meshes/wheel_4_1.stl" scale="0.001 0.001 0.001"/>
-    </geometry>
-    <material name="silver"/>
-  </visual>
-  <collision>
-    <origin xyz="-0.0 -0.0 0.025" rpy="0 0 0"/>
-    <geometry>
-      <mesh filename="file://$(find alphabot_description)/meshes/wheel_4_1.stl" scale="0.001 0.001 0.001"/>
+      <mesh filename="file://$(find atom_description)/meshes/wheel_4_1.stl" scale="0.001 0.001 0.001"/>
+    </geometry>
+    <material name="silver"/>
+  </visual>
+  <collision>
+    <origin xyz="-0.0 -0.0 0.025" rpy="0 0 0"/>
+    <geometry>
+      <mesh filename="file://$(find atom_description)/meshes/wheel_4_1.stl" scale="0.001 0.001 0.001"/>
     </geometry>
   </collision>
@@ -193,5 +193,5 @@
     <origin xyz="-0.0 -0.144399 -0.09" rpy="0 0 0"/>
     <geometry>
-      <mesh filename="file://$(find alphabot_description)/meshes/depth_camera_1.stl" scale="0.001 0.001 0.001"/>
+      <mesh filename="file://$(find atom_description)/meshes/depth_camera_1.stl" scale="0.001 0.001 0.001"/>
     </geometry>
     <material name="silver"/>
@@ -200,5 +200,5 @@
     <origin xyz="-0.0 -0.144399 -0.09" rpy="0 0 0"/>
     <geometry>
-      <mesh filename="file://$(find alphabot_description)/meshes/depth_camera_1.stl" scale="0.001 0.001 0.001"/>
+      <mesh filename="file://$(find atom_description)/meshes/depth_camera_1.stl" scale="0.001 0.001 0.001"/>
     </geometry>
   </collision>

File: alphabot_description/urdf/materials.xacro (robot description, xacro)
@@ -1,4 +1,4 @@
 <?xml version="1.0" ?>
-<robot name="alphabot" xmlns:xacro="http://www.ros.org/wiki/xacro" >
+<robot name="atom" xmlns:xacro="http://www.ros.org/wiki/xacro" >
 <material name="silver">
   <color rgba="0.700 0.700 0.700 1.000"/>
