Commit message: updated urdf files

File: atom_description/urdf/atom.xacro (robot description, xacro)
@@ -46,10 +46,10 @@
 <link name="wheel_1_1">
   <inertial>
-    <origin xyz="-0.06940433730274503 0.13399998634297935 2.287040556936404e-09" rpy="0 0 0"/>
+    <origin xyz="0.01859566269725499 -1.3657020569990408e-08 2.287040556936404e-09" rpy="0 0 0"/>
     <mass value="0.2827149727810706"/>
     <inertia ixx="0.000365" iyy="0.000217" izz="0.000217" ixy="0.0" iyz="0.0" ixz="-0.0"/>
   </inertial>
   <visual>
-    <origin xyz="-0.23 0.268 0.025" rpy="0 0 0"/>
+    <origin xyz="-0.14 0.134 0.025" rpy="0 0 0"/>
     <geometry>
       <mesh filename="file://$(find atom_description)/meshes/wheel_1_1.stl" scale="0.001 0.001 0.001"/>
@@ -58,5 +58,5 @@
   </visual>
   <collision>
-    <origin xyz="-0.23 0.268 0.025" rpy="0 0 0"/>
+    <origin xyz="-0.14 0.134 0.025" rpy="0 0 0"/>
     <geometry>
       <mesh filename="file://$(find atom_description)/meshes/wheel_1_1.stl" scale="0.001 0.001 0.001"/>
@@ -86,10 +86,10 @@
 <link name="wheel_2_1">
   <inertial>
-    <origin xyz="-0.06940433730274503 -0.1340000043103451 -1.3159243795329845e-08" rpy="0 0 0"/>
+    <origin xyz="0.01859566269725499 -4.3103450531045695e-09 -1.3159243784921504e-08" rpy="0 0 0"/>
     <mass value="0.2827149727810706"/>
     <inertia ixx="0.000365" iyy="0.000217" izz="0.000217" ixy="0.0" iyz="-0.0" ixz="0.0"/>
   </inertial>
   <visual>
-    <origin xyz="-0.23 -0.268 0.025" rpy="0 0 0"/>
+    <origin xyz="-0.14 -0.134 0.025" rpy="0 0 0"/>
     <geometry>
       <mesh filename="file://$(find atom_description)/meshes/wheel_2_1.stl" scale="0.001 0.001 0.001"/>
@@ -98,5 +98,5 @@
   </visual>
   <collision>
-    <origin xyz="-0.23 -0.268 0.025" rpy="0 0 0"/>
+    <origin xyz="-0.14 -0.134 0.025" rpy="0 0 0"/>
     <geometry>
       <mesh filename="file://$(find atom_description)/meshes/wheel_2_1.stl" scale="0.001 0.001 0.001"/>
@@ -146,10 +146,10 @@
 <link name="wheel_3_1">
   <inertial>
-    <origin xyz="-0.16059566269725498 -0.13400001370069212 2.0089295296732423e-09" rpy="0 0 0"/>
-    <mass value="0.2827149727810706"/>
-    <inertia ixx="0.000365" iyy="0.000217" izz="0.000217" ixy="-0.0" iyz="-0.0" ixz="0.0"/>
-  </inertial>
-  <visual>
-    <origin xyz="-0.0 -0.0 0.025" rpy="0 0 0"/>
+    <origin xyz="-0.01859566269725496 -1.3812480492703116e-08 -9.798722146181493e-10" rpy="0 0 0"/>
+    <mass value="0.2827149727810706"/>
+    <inertia ixx="0.000365" iyy="0.000217" izz="0.000217" ixy="-0.0" iyz="-0.0" ixz="-0.0"/>
+  </inertial>
+  <visual>
+    <origin xyz="0.14 0.134 0.025" rpy="0 0 0"/>
     <geometry>
       <mesh filename="file://$(find atom_description)/meshes/wheel_3_1.stl" scale="0.001 0.001 0.001"/>
@@ -158,5 +158,5 @@
   </visual>
   <collision>
-    <origin xyz="-0.0 -0.0 0.025" rpy="0 0 0"/>
+    <origin xyz="0.14 0.134 0.025" rpy="0 0 0"/>
     <geometry>
       <mesh filename="file://$(find atom_description)/meshes/wheel_3_1.stl" scale="0.001 0.001 0.001"/>
@@ -166,10 +166,10 @@
 <link name="wheel_4_1">
   <inertial>
-    <origin xyz="-0.1605956626972549 0.1339999861528064 4.9019815984152615e-14" rpy="0 0 0"/>
+    <origin xyz="-0.018595662697254906 -1.3847193641725042e-08 4.9384107914107744e-14" rpy="0 0 0"/>
     <mass value="0.2827149727810706"/>
     <inertia ixx="0.000365" iyy="0.000217" izz="0.000217" ixy="-0.0" iyz="-0.0" ixz="-0.0"/>
   </inertial>
   <visual>
-    <origin xyz="-0.0 -0.0 0.025" rpy="0 0 0"/>
+    <origin xyz="0.14 -0.134 0.025" rpy="0 0 0"/>
     <geometry>
       <mesh filename="file://$(find atom_description)/meshes/wheel_4_1.stl" scale="0.001 0.001 0.001"/>
@@ -178,5 +178,5 @@
   </visual>
   <collision>
-    <origin xyz="-0.0 -0.0 0.025" rpy="0 0 0"/>
+    <origin xyz="0.14 -0.134 0.025" rpy="0 0 0"/>
     <geometry>
       <mesh filename="file://$(find atom_description)/meshes/wheel_4_1.stl" scale="0.001 0.001 0.001"/>
@@ -210,5 +210,5 @@
 </joint>
 <joint name="wheel_clamp_1_to_wheel_1" type="continuous">
-  <origin xyz="0.115 -0.134 -0.085" rpy="0 0 0"/>
+  <origin xyz="0.025 0.0 -0.085" rpy="0 0 0"/>
   <parent link="wheel_clamp_1_1"/>
   <child link="wheel_1_1"/>
@@ -221,5 +221,5 @@
 </joint>
 <joint name="wheel_clamp_2_to_wheel_2" type="continuous">
-  <origin xyz="0.115 0.134 -0.085" rpy="0 0 0"/>
+  <origin xyz="0.025 0.0 -0.085" rpy="0 0 0"/>
   <parent link="wheel_clamp_2_1"/>
   <child link="wheel_2_1"/>
@@ -237,5 +237,5 @@
 </joint>
 <joint name="wheel_clamp_3_to_wheel_3" type="continuous">
-  <origin xyz="0.115 0.134 -0.085" rpy="0 0 0"/>
+  <origin xyz="-0.025 0.0 -0.085" rpy="0 0 0"/>
   <parent link="wheel_clamp_3_1"/>
   <child link="wheel_3_1"/>
@@ -243,5 +243,5 @@
 </joint>
 <joint name="wheel_clamp_4_to_wheel_4" type="continuous">
-  <origin xyz="0.115 -0.134 -0.085" rpy="0 0 0"/>
+  <origin xyz="-0.025 0.0 -0.085" rpy="0 0 0"/>
   <parent link="wheel_clamp_4_1"/>
   <child link="wheel_4_1"/>

Commit message: updated urdf

File: atom_description/urdf/atom.xacro (robot description, xacro)
@@ -44,24 +44,4 @@
   </collision>
 </link>
-<link name="wheel_1_1">
-  <inertial>
-    <origin xyz="0.01859566269725499 -1.3657020569990408e-08 2.287040556936404e-09" rpy="0 0 0"/>
-    <mass value="0.2827149727810706"/>
-    <inertia ixx="0.000365" iyy="0.000217" izz="0.000217" ixy="0.0" iyz="0.0" ixz="-0.0"/>
-  </inertial>
-  <visual>
-    <origin xyz="-0.14 0.134 0.025" rpy="0 0 0"/>
-    <geometry>
-      <mesh filename="file://$(find atom_description)/meshes/wheel_1_1.stl" scale="0.001 0.001 0.001"/>
-    </geometry>
-    <material name="silver"/>
-  </visual>
-  <collision>
-    <origin xyz="-0.14 0.134 0.025" rpy="0 0 0"/>
-    <geometry>
-      <mesh filename="file://$(find atom_description)/meshes/wheel_1_1.stl" scale="0.001 0.001 0.001"/>
-    </geometry>
-  </collision>
-</link>
 <link name="wheel_clamp_2_1">
   <inertial>
@@ -86,6 +66,6 @@
 <link name="wheel_2_1">
   <inertial>
-    <origin xyz="0.01859566269725499 -4.3103450531045695e-09 -1.3159243784921504e-08" rpy="0 0 0"/>
-    <mass value="0.2827149727810706"/>
+    <origin xyz="0.01859566269725499 -4.310345025348994e-09 -1.3159243767574269e-08" rpy="0 0 0"/>
+    <mass value="0.2827149727810705"/>
     <inertia ixx="0.000365" iyy="0.000217" izz="0.000217" ixy="0.0" iyz="-0.0" ixz="0.0"/>
   </inertial>
@@ -146,6 +126,6 @@
 <link name="wheel_3_1">
   <inertial>
-    <origin xyz="-0.01859566269725496 -1.3812480492703116e-08 -9.798722146181493e-10" rpy="0 0 0"/>
-    <mass value="0.2827149727810706"/>
+    <origin xyz="-0.01859566269725499 -1.3812480492703116e-08 -9.798722042098085e-10" rpy="0 0 0"/>
+    <mass value="0.2827149727810705"/>
     <inertia ixx="0.000365" iyy="0.000217" izz="0.000217" ixy="-0.0" iyz="-0.0" ixz="-0.0"/>
   </inertial>
@@ -166,6 +146,6 @@
 <link name="wheel_4_1">
   <inertial>
-    <origin xyz="-0.018595662697254906 -1.3847193641725042e-08 4.9384107914107744e-14" rpy="0 0 0"/>
-    <mass value="0.2827149727810706"/>
+    <origin xyz="-0.018595662697254906 -1.3847193613969466e-08 4.9394516254963605e-14" rpy="0 0 0"/>
+    <mass value="0.2827149727810705"/>
     <inertia ixx="0.000365" iyy="0.000217" izz="0.000217" ixy="-0.0" iyz="-0.0" ixz="-0.0"/>
   </inertial>
@@ -204,14 +184,28 @@
   </collision>
 </link>
+<link name="wheel_1_1">
+  <inertial>
+    <origin xyz="0.018595662697255044 -1.3159243611449156e-08 4.3103448345294115e-09" rpy="0 0 0"/>
+    <mass value="0.2827149727810706"/>
+    <inertia ixx="0.000365" iyy="0.000217" izz="0.000217" ixy="0.0" iyz="0.0" ixz="-0.0"/>
+  </inertial>
+  <visual>
+    <origin xyz="-0.14 0.134 0.025" rpy="0 0 0"/>
+    <geometry>
+      <mesh filename="file://$(find atom_description)/meshes/wheel_1_1.stl" scale="0.001 0.001 0.001"/>
+    </geometry>
+    <material name="silver"/>
+  </visual>
+  <collision>
+    <origin xyz="-0.14 0.134 0.025" rpy="0 0 0"/>
+    <geometry>
+      <mesh filename="file://$(find atom_description)/meshes/wheel_1_1.stl" scale="0.001 0.001 0.001"/>
+    </geometry>
+  </collision>
+</link>
 <joint name="base_link_to_wheel_clamp_1" type="fixed">
   <origin xyz="0.115 -0.134 0.06" rpy="0 0 0"/>
   <parent link="base_link"/>
   <child link="wheel_clamp_1_1"/>
-</joint>
-<joint name="wheel_clamp_1_to_wheel_1" type="continuous">
-  <origin xyz="0.025 0.0 -0.085" rpy="0 0 0"/>
-  <parent link="wheel_clamp_1_1"/>
-  <child link="wheel_1_1"/>
-  <axis xyz="1.0 0.0 0.0"/>
 </joint>
 <joint name="base_link_to_wheel_clamp_2" type="fixed">
@@ -253,3 +247,9 @@
   <child link="depth_camera_1"/>
 </joint>
+<joint name="Revolute 12" type="continuous">
+  <origin xyz="0.025 0.0 -0.085" rpy="0 0 0"/>
+  <parent link="wheel_clamp_1_1"/>
+  <child link="wheel_1_1"/>
+  <axis xyz="1.0 0.0 0.0"/>
+</joint>
 </robot>

Commit message: updated joint name

File: atom_description/urdf/atom.xacro (robot description, xacro)
@@ -44,4 +44,24 @@
   </collision>
 </link>
+<link name="wheel_1_1">
+  <inertial>
+    <origin xyz="0.01859566269725499 -1.3657020569990408e-08 2.287040556936404e-09" rpy="0 0 0"/>
+    <mass value="0.2827149727810706"/>
+    <inertia ixx="0.000365" iyy="0.000217" izz="0.000217" ixy="0.0" iyz="0.0" ixz="-0.0"/>
+  </inertial>
+  <visual>
+    <origin xyz="-0.14 0.134 0.025" rpy="0 0 0"/>
+    <geometry>
+      <mesh filename="file://$(find atom_description)/meshes/wheel_1_1.stl" scale="0.001 0.001 0.001"/>
+    </geometry>
+    <material name="silver"/>
+  </visual>
+  <collision>
+    <origin xyz="-0.14 0.134 0.025" rpy="0 0 0"/>
+    <geometry>
+      <mesh filename="file://$(find atom_description)/meshes/wheel_1_1.stl" scale="0.001 0.001 0.001"/>
+    </geometry>
+  </collision>
+</link>
 <link name="wheel_clamp_2_1">
   <inertial>
@@ -66,6 +86,6 @@
 <link name="wheel_2_1">
   <inertial>
-    <origin xyz="0.01859566269725499 -4.310345025348994e-09 -1.3159243767574269e-08" rpy="0 0 0"/>
-    <mass value="0.2827149727810705"/>
+    <origin xyz="0.01859566269725499 -4.3103450531045695e-09 -1.3159243784921504e-08" rpy="0 0 0"/>
+    <mass value="0.2827149727810706"/>
     <inertia ixx="0.000365" iyy="0.000217" izz="0.000217" ixy="0.0" iyz="-0.0" ixz="0.0"/>
   </inertial>
@@ -126,6 +146,6 @@
 <link name="wheel_3_1">
   <inertial>
-    <origin xyz="-0.01859566269725499 -1.3812480492703116e-08 -9.798722042098085e-10" rpy="0 0 0"/>
-    <mass value="0.2827149727810705"/>
+    <origin xyz="-0.01859566269725496 -1.3812480492703116e-08 -9.798722146181493e-10" rpy="0 0 0"/>
+    <mass value="0.2827149727810706"/>
     <inertia ixx="0.000365" iyy="0.000217" izz="0.000217" ixy="-0.0" iyz="-0.0" ixz="-0.0"/>
   </inertial>
@@ -146,6 +166,6 @@
 <link name="wheel_4_1">
   <inertial>
-    <origin xyz="-0.018595662697254906 -1.3847193613969466e-08 4.9394516254963605e-14" rpy="0 0 0"/>
-    <mass value="0.2827149727810705"/>
+    <origin xyz="-0.018595662697254906 -1.3847193641725042e-08 4.9384107914107744e-14" rpy="0 0 0"/>
+    <mass value="0.2827149727810706"/>
     <inertia ixx="0.000365" iyy="0.000217" izz="0.000217" ixy="-0.0" iyz="-0.0" ixz="-0.0"/>
   </inertial>
@@ -184,28 +204,14 @@
   </collision>
 </link>
-<link name="wheel_1_1">
-  <inertial>
-    <origin xyz="0.018595662697255044 -1.3159243611449156e-08 4.3103448345294115e-09" rpy="0 0 0"/>
-    <mass value="0.2827149727810706"/>
-    <inertia ixx="0.000365" iyy="0.000217" izz="0.000217" ixy="0.0" iyz="0.0" ixz="-0.0"/>
-  </inertial>
-  <visual>
-    <origin xyz="-0.14 0.134 0.025" rpy="0 0 0"/>
-    <geometry>
-      <mesh filename="file://$(find atom_description)/meshes/wheel_1_1.stl" scale="0.001 0.001 0.001"/>
-    </geometry>
-    <material name="silver"/>
-  </visual>
-  <collision>
-    <origin xyz="-0.14 0.134 0.025" rpy="0 0 0"/>
-    <geometry>
-      <mesh filename="file://$(find atom_description)/meshes/wheel_1_1.stl" scale="0.001 0.001 0.001"/>
-    </geometry>
-  </collision>
-</link>
 <joint name="base_link_to_wheel_clamp_1" type="fixed">
   <origin xyz="0.115 -0.134 0.06" rpy="0 0 0"/>
   <parent link="base_link"/>
   <child link="wheel_clamp_1_1"/>
+</joint>
+<joint name="wheel_clamp_1_to_wheel_1" type="continuous">
+  <origin xyz="0.025 0.0 -0.085" rpy="0 0 0"/>
+  <parent link="wheel_clamp_1_1"/>
+  <child link="wheel_1_1"/>
+  <axis xyz="1.0 0.0 0.0"/>
 </joint>
 <joint name="base_link_to_wheel_clamp_2" type="fixed">
@@ -247,9 +253,3 @@
   <child link="depth_camera_1"/>
 </joint>
-<joint name="Revolute 12" type="continuous">
-  <origin xyz="0.025 0.0 -0.085" rpy="0 0 0"/>
-  <parent link="wheel_clamp_1_1"/>
-  <child link="wheel_1_1"/>
-  <axis xyz="1.0 0.0 0.0"/>
-</joint>
 </robot>
