Commit message: updated folder layout

File: src/atom_description/urdf/atom.xacro (robot description, xacro)
@@ -55,5 +55,5 @@
       <mesh filename="file://$(find atom_description)/meshes/wheel_1_1.stl" scale="0.001 0.001 0.001"/>
     </geometry>
-    <material name="silver"/>
+    <material name="black" />
   </visual>
   <collision>
@@ -95,5 +95,5 @@
       <mesh filename="file://$(find atom_description)/meshes/wheel_2_1.stl" scale="0.001 0.001 0.001"/>
     </geometry>
-    <material name="silver"/>
+    <material name="black" />
   </visual>
   <collision>
@@ -155,5 +155,5 @@
       <mesh filename="file://$(find atom_description)/meshes/wheel_3_1.stl" scale="0.001 0.001 0.001"/>
     </geometry>
-    <material name="silver"/>
+    <material name="black" />
   </visual>
   <collision>
@@ -175,5 +175,5 @@
       <mesh filename="file://$(find atom_description)/meshes/wheel_4_1.stl" scale="0.001 0.001 0.001"/>
     </geometry>
-    <material name="silver"/>
+    <material name="black" />
   </visual>
   <collision>

File: src/atom_description/urdf/materials.xacro (robot description, xacro)
@@ -4,3 +4,6 @@
   <color rgba="0.700 0.700 0.700 1.000"/>
 </material>
+<material name="black">
+  <color rgba="0 0 0 1"/>
+</material>
 </robot>
