Commit message: created the robot with 4 wheeled diff drive support

File: src/atom_description/.urdf/atom.xacro (robot description, xacro)
@@ -7,9 +7,4 @@
 <xacro:include filename="$(find atom_description)/urdf/plugins.xacro" />
 <link name="base_link">
-  <inertial>
-    <origin xyz="-1.0547369564692681e-07 0.004021237681352332 0.0412312225257285" rpy="0 0 0"/>
-    <mass value="8.373395552650207"/>
-    <inertia ixx="0.115141" iyy="0.045372" izz="0.151049" ixy="0.0" iyz="-0.001432" ixz="-0.0"/>
-  </inertial>
   <visual>
     <origin xyz="0 0 0" rpy="0 0 0"/>

File: src/atom_description/.urdf/plugins.xacro (robot description, xacro)
@@ -10,6 +10,8 @@
       <right_joint>wheel_clamp_1_to_wheel_1</right_joint>
       <left_joint>wheel_clamp_3_to_wheel_3</left_joint>
+      <!-- <right_joint>wheel_clamp_2_to_wheel_2</right_joint>
+      <left_joint>wheel_clamp_4_to_wheel_4</left_joint> -->
       <!-- kinematics -->
-      <wheel_separation>0.280</wheel_separation>
+      <wheel_separation>0.340</wheel_separation>
       <wheel_diameter>0.100</wheel_diameter>
       <!-- limits -->
