Commit message: updated robots

File: src/atom_description/old_urdf/atom.xacro (robot description, xacro)
@@ -1,9 +1,9 @@
 <?xml version="1.0" ?>
 <robot name="atom" xmlns:xacro="http://www.ros.org/wiki/xacro">
-<xacro:include filename="$(find atom_description)/urdf/materials.xacro" />
-<xacro:include filename="$(find atom_description)/urdf/atom.trans" />
-<xacro:include filename="$(find atom_description)/urdf/atom.gazebo" />
-<!-- <xacro:include filename="$(find atom_description)/urdf/base_footprint.xacro" /> -->
-<xacro:include filename="$(find atom_description)/urdf/plugins.xacro" />
+<xacro:include filename="$(find atom_description)/old_urdf/materials.xacro" />
+<xacro:include filename="$(find atom_description)/old_urdf/atom.trans" />
+<xacro:include filename="$(find atom_description)/old_urdf/atom.gazebo" />
+<xacro:include filename="$(find atom_description)/old_urdf/base_footprint.xacro" />
+<xacro:include filename="$(find atom_description)/old_urdf/plugins.xacro" />
 <link name="base_link">
   <visual>
@@ -237,5 +237,5 @@
   <parent link="wheel_clamp_3_1"/>
   <child link="wheel_3_1"/>
-  <axis xyz="-1.0 0.0 -0.0"/>
+  <axis xyz="1.0 0.0 0.0"/>
 </joint>
 <joint name="wheel_clamp_4_to_wheel_4" type="continuous">
@@ -243,5 +243,5 @@
   <parent link="wheel_clamp_4_1"/>
   <child link="wheel_4_1"/>
-  <axis xyz="-1.0 0.0 0.0"/>
+  <axis xyz="1.0 0.0 0.0"/>
 </joint>
 <joint name="base_link_to_depth_camera" type="fixed">

File: src/atom_description/old_urdf/materials.xacro (robot description, xacro)
@@ -2,8 +2,8 @@
 <robot name="atom" xmlns:xacro="http://www.ros.org/wiki/xacro" >
 <material name="silver">
-  <color rgba="0.700 0.700 0.700 1.000"/>
+  <color rgba="0.700 0.700 0.700 0.5"/>
 </material>
 <material name="black">
-  <color rgba="0 0 0 1"/>
+  <color rgba="0 0 0 0.5"/>
 </material>
 </robot>

File: src/atom_description/old_urdf/plugins.xacro (robot description, xacro)
@@ -7,15 +7,20 @@
       <!-- Update rate in Hz -->
       <update_rate>50</update_rate>
+      <num_wheel_pairs>2</num_wheel_pairs>
       <!-- wheels -->
+      <left_joint>wheel_clamp_3_to_wheel_3</left_joint>
       <right_joint>wheel_clamp_1_to_wheel_1</right_joint>
-      <left_joint>wheel_clamp_3_to_wheel_3</left_joint>
-      <!-- <right_joint>wheel_clamp_2_to_wheel_2</right_joint>
-      <left_joint>wheel_clamp_4_to_wheel_4</left_joint> -->
+      <left_joint>wheel_clamp_4_to_wheel_4</left_joint>
+      <right_joint>wheel_clamp_2_to_wheel_2</right_joint>
       <!-- kinematics -->
-      <wheel_separation>0.340</wheel_separation>
+       <!-- 0.7 + 2*0.01  -->
+      <wheel_separation>0.280</wheel_separation>
+      <wheel_separation>0.72</wheel_separation>
+      <!-- 0.13 * 2 -->
+      <wheel_diameter>0.26</wheel_diameter>
       <wheel_diameter>0.100</wheel_diameter>
       <!-- limits -->
-      <!-- <max_wheel_torque>20</max_wheel_torque>
-      <max_wheel_acceleration>1.0</max_wheel_acceleration> -->
+      <max_wheel_torque>20</max_wheel_torque>
+      <max_wheel_acceleration>1.0</max_wheel_acceleration>
       <!-- input -->
       <command_topic>cmd_vel</command_topic>

File: src/atom_description/urdf/atom.gazebo.urdf.xacro (robot description, xacro)
@@ -16,3 +16,6 @@
         <material>Gazebo/Black</material>
     </gazebo>
+    <gazebo reference="camera">
+        <material>Gazebo/Black</material>
+    </gazebo>
 </robot>

File: src/atom_description/urdf/atom.urdf.xacro (robot description, xacro)
@@ -4,4 +4,5 @@
     <xacro:include filename="$(find atom_description)/urdf/common.urdf.xacro" />
     <xacro:include filename="$(find atom_description)/urdf/robot.urdf.xacro" />
+    <xacro:include filename="$(find atom_description)/urdf/camera.plugin.urdf.xacro" />
     <xacro:include filename="$(find atom_description)/urdf/atom.gazebo.urdf.xacro" />
     <xacro:include filename="$(find atom_description)/urdf/plugins.urdf.xacro" />

File: src/atom_description/urdf/common.urdf.xacro (robot description, xacro)
@@ -3,4 +3,7 @@
     <material name="black">
         <color rgba="0 0 0 0.75" />
+    </material>
+    <material name="white">
+        <color rgba="1 1 1 0.75" />
     </material>
     <material name="red">

File: src/atom_description/urdf/variables.urdf.xacro (robot description, xacro)
@@ -10,4 +10,7 @@
     <xacro:property name="wheel_distance_from_base" value="${ wheel_radius - 0.05 }" />
     <xacro:property name="base_footprint_to_base_link_distance" value="${wheel_distance_from_base + wheel_radius}" />
+    <xacro:property name="camera_length" value="0.02" />
+    <xacro:property name="camera_width" value="0.10" />
+    <xacro:property name="camera_height" value="0.06" />
     <xacro:property name="xyz_base_link_to_front_left_wheel" value="${ (base_length / 2) - wheel_radius } ${ (base_width / 2) + buffer_space_for_wheels } ${ -wheel_distance_from_base }" />
     <xacro:property name="xyz_base_link_to_front_right_wheel" value="${ (base_length / 2) - wheel_radius } ${ -((base_width / 2) + buffer_space_for_wheels) } ${ -wheel_distance_from_base }" />
