Commit message: updated line follower with CV

File: src/line_follower_description/robot_urdf/camera.xacro (robot description, xacro)
@@ -19,8 +19,8 @@
                     <!-- <format>R8G8B8</format> -->
                 </image>
+               <update_rate>30.0</update_rate>
             </camera>
             <pose>0 0 0 0 0 0</pose>
             <visualize>true</visualize>
-            <update_rate>30.0</update_rate>
             <!-- <camera></camera> -->
             <plugin name="camera_controller" filename="libgazebo_ros_camera.so">

File: src/line_follower_description/robot_urdf/plugins.xacro (robot description, xacro)
@@ -1,6 +1,6 @@
 <?xml version="1.0"?>
 <robot name="line_follower" xmlns:xacro="http://www.ros.org/wiki/xacro">
-  <xacro:property name="wheel_separation" value="0.280"/>
-  <xacro:property name="wheel_diameter" value="0.100"/>
+  <xacro:property name="wheel_separation" value="0.280" />
+  <xacro:property name="wheel_diameter" value="0.100" />
   <gazebo>
     <plugin name="diff_drive_controller" filename="libgazebo_ros_diff_drive.so">
@@ -14,5 +14,5 @@
       <right_joint>wheel_clamp_1_to_wheel_1</right_joint>
       <!-- kinematics -->
-       <!-- 0.7 + 2*0.01  -->
+      <!-- 0.7 + 2*0.01  -->
       <wheel_separation>0.280</wheel_separation>
       <wheel_separation>0.280</wheel_separation>
